Commit message: gazeebo autonomous vehicle

File: qcar_docker/qcar/rosws/src/qcar_description/urdf/qcar.gazebo.xacro (robot description, xacro)
@@ -1,11 +1,14 @@
 <?xml version="1.0"?>
 <robot name="QCar" xmlns:xacro="http://www.ros.org/wiki/xacro">
-<!-- Define all the computer vision sernsor properties -->
-	<gazebo reference="camera_rgb">
-    <!-- <material>Gazebo/Green</material> -->
+<!-- ROS 2 Gazebo Plugins for QCar -->
+  <!-- Base link must have inertia for Gazebo -->
+  <gazebo reference="base">
+    <material>Gazebo/Orange</material>
+  </gazebo>
+  <!-- RGB Camera (Intel RealSense) - ROS 2 -->
+  <gazebo reference="camera_rgb">
     <sensor type="camera" name="intelrealsense_rgb">
-    	<pose>0 0 0 0 0 0</pose>
-    	<!-- <pose>0.081686 0.031547 0.15445 0 0 0</pose> -->
-      <update_rate>60.0</update_rate>
+      <pose>0 0 0 0 0 0</pose>
+      <update_rate>30.0</update_rate>
       <camera name="rgb">
         <horizontal_fov>1.21126</horizontal_fov>
@@ -21,25 +24,20 @@
       </camera>
       <plugin name="camera_controller" filename="libgazebo_ros_camera.so">
-        <alwaysOn>true</alwaysOn>
-        <updateRate>0.0</updateRate>
-        <cameraName>qcar/rgb</cameraName>
-        <imageTopicName>image_color</imageTopicName>
-        <cameraInfoTopicName>camera_info</cameraInfoTopicName>
-        <frameName>camera_rgb</frameName>
-        <hackBaseline>0.07</hackBaseline>
-        <distortionK1>0.0</distortionK1>
-        <distortionK2>0.0</distortionK2>
-        <distortionK3>0.0</distortionK3>
-        <distortionT1>0.0</distortionT1>
-        <distortionT2>0.0</distortionT2>
-      </plugin>
-    </sensor>
-  </gazebo>
+        <ros>
+          <namespace>qcar</namespace>
+          <remapping>image_raw:=rgb/image_color</remapping>
+          <remapping>camera_info:=rgb/camera_info</remapping>
+        </ros>
+        <camera_name>rgb</camera_name>
+        <frame_name>camera_rgb</frame_name>
+        <hack_baseline>0.07</hack_baseline>
+      </plugin>
+    </sensor>
+  </gazebo>
+  <!-- CSI Front Camera - ROS 2 -->
   <gazebo reference="camera_csi_front">
-    <!-- <material>Gazebo/Green</material> -->
     <sensor type="camera" name="csi_front">
-    	<pose>0 0 0 0 0 0</pose>
-    	<!-- <pose>0.081686 0.031547 0.15445 0 0 0</pose> -->
-      <update_rate>60.0</update_rate>
+      <pose>0 0 0 0 0 0</pose>
+      <update_rate>30.0</update_rate>
       <camera name="front">
         <horizontal_fov>2.79253</horizontal_fov>
@@ -53,27 +51,28 @@
           <far>300</far>
         </clip>
-      </camera>
-      <plugin name="camera_controller" filename="libgazebo_ros_camera.so">
-        <alwaysOn>true</alwaysOn>
-        <updateRate>0.0</updateRate>
-        <cameraName>qcar/csi_front</cameraName>
-        <imageTopicName>image_raw</imageTopicName>
-        <cameraInfoTopicName>camera_info</cameraInfoTopicName>
-        <frameName>camera_csi_front</frameName>
-        <hackBaseline>0.07</hackBaseline>
-        <distortionK1>-0.264598808</distortionK1>
-        <distortionK2>0.0156281135</distortionK2>
-        <distortionK3>0.0822019378</distortionK3>
-        <distortionT1>0.0000652954</distortionT1>
-        <distortionT2>0.0053984313</distortionT2>
-      </plugin>
-    </sensor>
-  </gazebo>
+        <distortion>
+          <k1>-0.264598808</k1>
+          <k2>0.0156281135</k2>
+          <k3>0.0822019378</k3>
+          <p1>0.0000652954</p1>
+          <p2>0.0053984313</p2>
+        </distortion>
+      </camera>
+      <plugin name="camera_csi_front_controller" filename="libgazebo_ros_camera.so">
+        <ros>
+          <namespace>qcar</namespace>
+          <remapping>image_raw:=csi_front/image_raw</remapping>
+          <remapping>camera_info:=csi_front/camera_info</remapping>
+        </ros>
+        <camera_name>csi_front</camera_name>
+        <frame_name>camera_csi_front</frame_name>
+      </plugin>
+    </sensor>
+  </gazebo>
+  <!-- CSI Right Camera - ROS 2 -->
   <gazebo reference="camera_csi_right">
-    <!-- <material>Gazebo/Green</material> -->
     <sensor type="camera" name="csi_right">
-    	<pose>0 0 0 0 0 0</pose>
-    	<!-- <pose>0.081686 0.031547 0.15445 0 0 0</pose> -->
-      <update_rate>60.0</update_rate>
+      <pose>0 0 0 0 0 0</pose>
+      <update_rate>30.0</update_rate>
       <camera name="right">
         <horizontal_fov>2.79253</horizontal_fov>
@@ -87,27 +86,28 @@
           <far>300</far>
         </clip>
-      </camera>
-      <plugin name="camera_controller" filename="libgazebo_ros_camera.so">
-        <alwaysOn>true</alwaysOn>
-        <updateRate>0.0</updateRate>
-        <cameraName>qcar/csi_right</cameraName>
-        <imageTopicName>image_raw</imageTopicName>
-        <cameraInfoTopicName>camera_info</cameraInfoTopicName>
-        <frameName>camera_csi_right</frameName>
-        <hackBaseline>0.07</hackBaseline>
-       	<distortionK1>-0.264598808</distortionK1>
-        <distortionK2>0.0156281135</distortionK2>
-        <distortionK3>0.0822019378</distortionK3>
-        <distortionT1>0.0000652954</distortionT1>
-        <distortionT2>0.0053984313</distortionT2>
-      </plugin>
-    </sensor>
-  </gazebo>
+        <distortion>
+          <k1>-0.264598808</k1>
+          <k2>0.0156281135</k2>
+          <k3>0.0822019378</k3>
+          <p1>0.0000652954</p1>
+          <p2>0.0053984313</p2>
+        </distortion>
+      </camera>
+      <plugin name="camera_csi_right_controller" filename="libgazebo_ros_camera.so">
+        <ros>
+          <namespace>qcar</namespace>
+          <remapping>image_raw:=csi_right/image_raw</remapping>
+          <remapping>camera_info:=csi_right/camera_info</remapping>
+        </ros>
+        <camera_name>csi_right</camera_name>
+        <frame_name>camera_csi_right</frame_name>
+      </plugin>
+    </sensor>
+  </gazebo>
+  <!-- CSI Back Camera - ROS 2 -->
   <gazebo reference="camera_csi_back">
-    <!-- <material>Gazebo/Green</material> -->
     <sensor type="camera" name="csi_back">
-    	<pose>0 0 0 0 0 0</pose>
-    	<!-- <pose>0.081686 0.031547 0.15445 0 0 0</pose> -->
-      <update_rate>60.0</update_rate>
+      <pose>0 0 0 0 0 0</pose>
+      <update_rate>30.0</update_rate>
       <camera name="back">
         <horizontal_fov>2.79253</horizontal_fov>
@@ -121,27 +121,28 @@
           <far>300</far>
         </clip>
-      </camera>
-      <plugin name="camera_controller" filename="libgazebo_ros_camera.so">
-        <alwaysOn>true</alwaysOn>
-        <updateRate>0.0</updateRate>
-        <cameraName>qcar/csi_back</cameraName>
-        <imageTopicName>image_raw</imageTopicName>
-        <cameraInfoTopicName>camera_info</cameraInfoTopicName>
-        <frameName>camera_csi_back</frameName>
-        <hackBaseline>0.07</hackBaseline>
-        <distortionK1>-0.264598808</distortionK1>
-        <distortionK2>0.0156281135</distortionK2>
-        <distortionK3>0.0822019378</distortionK3>
-        <distortionT1>0.0000652954</distortionT1>
-        <distortionT2>0.0053984313</distortionT2>
-      </plugin>
-    </sensor>
-  </gazebo>
+        <distortion>
+          <k1>-0.264598808</k1>
+          <k2>0.0156281135</k2>
+          <k3>0.0822019378</k3>
+          <p1>0.0000652954</p1>
+          <p2>0.0053984313</p2>
+        </distortion>
+      </camera>
+      <plugin name="camera_csi_back_controller" filename="libgazebo_ros_camera.so">
+        <ros>
+          <namespace>qcar</namespace>
+          <remapping>image_raw:=csi_back/image_raw</remapping>
+          <remapping>camera_info:=csi_back/camera_info</remapping>
+        </ros>
+        <camera_name>csi_back</camera_name>
+        <frame_name>camera_csi_back</frame_name>
+      </plugin>
+    </sensor>
+  </gazebo>
+  <!-- CSI Left Camera - ROS 2 -->
   <gazebo reference="camera_csi_left">
-    <!-- <material>Gazebo/Green</material> -->
     <sensor type="camera" name="csi_left">
-    	<pose>0 0 0 0 0 0</pose>
-    	<!-- <pose>0.081686 0.031547 0.15445 0 0 0</pose> -->
-      <update_rate>60.0</update_rate>
+      <pose>0 0 0 0 0 0</pose>
+      <update_rate>30.0</update_rate>
       <camera name="left">
         <horizontal_fov>2.79253</horizontal_fov>
@@ -155,32 +156,33 @@
           <far>300</far>
         </clip>
-      </camera>
-      <plugin name="camera_controller" filename="libgazebo_ros_camera.so">
-        <alwaysOn>true</alwaysOn>
-        <updateRate>0.0</updateRate>
-        <cameraName>qcar/csi_left</cameraName>
-        <imageTopicName>image_raw</imageTopicName>
-        <cameraInfoTopicName>camera_info</cameraInfoTopicName>
-        <frameName>camera_csi_left</frameName>
-        <hackBaseline>0.07</hackBaseline>
-        <distortionK1>-0.264598808</distortionK1>
-        <distortionK2>0.0156281135</distortionK2>
-        <distortionK3>0.0822019378</distortionK3>
-        <distortionT1>0.0000652954</distortionT1>
-        <distortionT2>0.0053984313</distortionT2>
-      </plugin>
-    </sensor>
-  </gazebo>
+        <distortion>
+          <k1>-0.264598808</k1>
+          <k2>0.0156281135</k2>
+          <k3>0.0822019378</k3>
+          <p1>0.0000652954</p1>
+          <p2>0.0053984313</p2>
+        </distortion>
+      </camera>
+      <plugin name="camera_csi_left_controller" filename="libgazebo_ros_camera.so">
+        <ros>
+          <namespace>qcar</namespace>
+          <remapping>image_raw:=csi_left/image_raw</remapping>
+          <remapping>camera_info:=csi_left/camera_info</remapping>
+        </ros>
+        <camera_name>csi_left</camera_name>
+        <frame_name>camera_csi_left</frame_name>
+      </plugin>
+    </sensor>
+  </gazebo>
+  <!-- LIDAR Sensor - ROS 2 -->
   <gazebo reference="lidar">
     <sensor type="ray" name="head_rplidar_sensor">
-      <pose>0 0 0.010 -0 0</pose>
+      <pose>0 0 0.010 0 0 0</pose>
       <visualize>true</visualize>
-      <!-- <visualize>false</visualize> -->
-      <alwaysOn>true</alwaysOn>
-      <update_rate>30</update_rate>
+      <update_rate>10</update_rate>
       <ray>
         <scan>
           <horizontal>
-            <samples>240</samples>
+            <samples>360</samples>
             <resolution>1</resolution>
             <min_angle>-3.14159</min_angle>
@@ -189,23 +191,86 @@
         </scan>
         <range>
-          <min>0.10</min>
+          <min>0.12</min>
           <max>12.0</max>
-          <resolution>0.01</resolution>
+          <resolution>0.015</resolution>
         </range>
         <noise>
           <type>gaussian</type>
-          <!-- Noise parameters based on published spec for Hokuyo laser
-               achieving "+-30mm" accuracy at range < 10m.  A mean of 0.0m and
-               stddev of 0.01m will put 99.7% of samples within 0.03m of the true
-               reading. -->
           <mean>0.0</mean>
           <stddev>0.01</stddev>
         </noise>
       </ray>
-      <plugin name="gazebo_ros_head_rplidar_controller" filename="libgazebo_ros_laser.so">
-        <topicName>/qcar/lidar</topicName>
-        <frameName>lidar</frameName>
-      </plugin>
-    </sensor>
+      <plugin name="gazebo_ros_rplidar" filename="libgazebo_ros_ray_sensor.so">
+        <ros>
+          <namespace>qcar</namespace>
+          <remapping>~/out:=lidar/scan</remapping>
+        </ros>
+        <output_type>sensor_msgs/LaserScan</output_type>
+        <frame_name>lidar</frame_name>
+      </plugin>
+    </sensor>
+  </gazebo>
+  <!-- Differential Drive Plugin for QCar - ROS 2 -->
+  <gazebo>
+    <plugin name="differential_drive_controller" filename="libgazebo_ros_diff_drive.so">
+      <ros>
+        <namespace>qcar</namespace>
+        <remapping>cmd_vel:=cmd_vel</remapping>
+        <remapping>odom:=odom</remapping>
+      </ros>
+      <!-- Wheel joints -->
+      <left_joint>left_rear_axle</left_joint>
+      <right_joint>right_rear_axle</right_joint>
+      <!-- Kinematics -->
+      <wheel_separation>0.112</wheel_separation>
+      <wheel_diameter>0.053</wheel_diameter>
+      <!-- Limits -->
+      <max_wheel_torque>2.0</max_wheel_torque>
+      <max_wheel_acceleration>1.0</max_wheel_acceleration>
+      <!-- Output -->
+      <publish_odom>true</publish_odom>
+      <publish_odom_tf>true</publish_odom_tf>
+      <publish_wheel_tf>false</publish_wheel_tf>
+      <odometry_frame>odom</odometry_frame>
+      <robot_base_frame>base_link</robot_base_frame>
+      <update_rate>50</update_rate>
+    </plugin>
+  </gazebo>
+  <!-- Ground plane contact for wheels -->
+  <gazebo reference="left_front_wheel">
+    <material>Gazebo/DarkGrey</material>
+    <mu1>1.0</mu1>
+    <mu2>1.0</mu2>
+    <kp>1000000.0</kp>
+    <kd>100.0</kd>
+    <minDepth>0.001</minDepth>
+    <maxVel>1.0</maxVel>
+  </gazebo>
+  <gazebo reference="right_front_wheel">
+    <material>Gazebo/DarkGrey</material>
+    <mu1>1.0</mu1>
+    <mu2>1.0</mu2>
+    <kp>1000000.0</kp>
+    <kd>100.0</kd>
+    <minDepth>0.001</minDepth>
+    <maxVel>1.0</maxVel>
+  </gazebo>
+  <gazebo reference="left_rear_wheel">
+    <material>Gazebo/DarkGrey</material>
+    <mu1>1.0</mu1>
+    <mu2>1.0</mu2>
+    <kp>1000000.0</kp>
+    <kd>100.0</kd>
+    <minDepth>0.001</minDepth>
+    <maxVel>1.0</maxVel>
+  </gazebo>
+  <gazebo reference="right_rear_wheel">
+    <material>Gazebo/DarkGrey</material>
+    <mu1>1.0</mu1>
+    <mu2>1.0</mu2>
+    <kp>1000000.0</kp>
+    <kd>100.0</kd>
+    <minDepth>0.001</minDepth>
+    <maxVel>1.0</maxVel>
   </gazebo>
 </robot>
